Commit message: 阿克曼模型建立和轮子修复

File: zebrat/urdf/R1.urdf (robot description, URDF)
Before this commit: robot R1, 10 links, 9 joints
Links:
- removed link base_footprint
- added link front_left_steering_link, mass 0.30
- added link front_right_steering_link, mass 0.30
- link Empty_Link1: geometry collision cylinder length=0.040 radius=0.04075; visual cylinder length=0.040 radius=0.04075
- link Empty_Link2: geometry collision cylinder length=0.040 radius=0.04075; visual cylinder length=0.040 radius=0.04075
- link Empty_Link3: geometry collision cylinder length=0.0465 radius=0.04075; visual cylinder length=0.0465 radius=0.04075
- link Empty_Link4: geometry collision cylinder length=0.0465 radius=0.04075; visual cylinder length=0.0465 radius=0.04075
- link base_link: geometry collision box size=0.50 0.16 0.22; visual mesh filename=package://zebrat/urdf/meshes/base_link.stl
Joints:
- removed joint J1
- removed joint J2
- removed joint J3
- removed joint J4
- removed joint base_footprint_joint
- added joint front_left_steering_joint: type revolute, parent base_link, child front_left_steering_link, origin xyz=0.220127909860013 0.142085316479216 0.04075 rpy=0 0 0, axis 0 0 1, limit lower=-0.6 upper=0.6 effort=30 velocity=4
- added joint front_left_wheel_joint: type continuous, parent front_left_steering_link, child Empty_Link1, origin xyz=0 0 -0.04075 rpy=0 0 0, axis 0 1 0, limit effort=30 velocity=60
- added joint front_right_steering_joint: type revolute, parent base_link, child front_right_steering_link, origin xyz=0.220127909860013 -0.122535316479216 0.04075 rpy=0 0 0, axis 0 0 1, limit lower=-0.6 upper=0.6 effort=30 velocity=4
- added joint front_right_wheel_joint: type continuous, parent front_right_steering_link, child Empty_Link2, origin xyz=0 0 -0.04075 rpy=0 0 0, axis 0 -1 0, limit effort=30 velocity=60
- added joint rear_left_wheel_joint: type continuous, parent base_link, child Empty_Link4, origin xyz=-0.19879978611665 0.119285316479219 0.0 rpy=0 0 0, axis 0 1 0, limit effort=20 velocity=20
- added joint rear_right_wheel_joint: type continuous, parent base_link, child Empty_Link3, origin xyz=-0.19879978611665 -0.122535316479219 0.0 rpy=0 0 0, axis 0 -1 0, limit effort=20 velocity=20

File: zebrat/urdf/R1_rviz.urdf (robot description, URDF)
Before this commit: robot R1_rviz, 10 links, 9 joints
Links:
- added link front_left_steering_link
- added link front_right_steering_link
Joints:
- removed joint J1
- removed joint J2
- removed joint J3
- removed joint J4
- added joint front_left_steering_joint: type revolute, parent base_link, child front_left_steering_link, origin xyz=0.220127909860013 0.142085316479216 0.04075 rpy=0 0 0, axis 0 0 1, limit lower=-0.6 upper=0.6 effort=30 velocity=4
- added joint front_left_wheel_joint: type continuous, parent front_left_steering_link, child Empty_Link1, origin xyz=0 0 -0.04075 rpy=0 0 0, axis 0 1 0
- added joint front_right_steering_joint: type revolute, parent base_link, child front_right_steering_link, origin xyz=0.220127909860013 -0.122535316479216 0.04075 rpy=0 0 0, axis 0 0 1, limit lower=-0.6 upper=0.6 effort=30 velocity=4
- added joint front_right_wheel_joint: type continuous, parent front_right_steering_link, child Empty_Link2, origin xyz=0 0 -0.04075 rpy=0 0 0, axis 0 -1 0
- added joint rear_left_wheel_joint: type continuous, parent base_link, child Empty_Link4, origin xyz=-0.19879978611665 0.119285316479219 0.0 rpy=0 0 0, axis 0 1 0
- added joint rear_right_wheel_joint: type continuous, parent base_link, child Empty_Link3, origin xyz=-0.19879978611665 -0.122535316479219 0.0 rpy=0 0 0, axis 0 -1 0
